File: HIGH-POWER-12V_Converter_LM51231-Q1/12V_Converter_LM5152x-Q1/12V_Converter_LM5152x-Q1.kicad_sch (KiCad schematic)
At the start: 30 parts, among them M1 60V, M2 60V, U1 LM51521QRGRRQ1

Commit message: added some jlcpcb pick n place files
Parts:
- Cbias1, Cbst1: LCSC (none) -> C92759
- Ccomp2: LCSC (none) -> C107111
- Cin1, Cin2, Coutx1, Coutx2, Coutx3, Coutx4, Coutx5, Coutx6, Coutx7, Coutx8: LCSC (none) -> C77093
- Cinx1: LCSC (none) -> C2172920
- Cvout1: LCSC (none) -> C2842861
- Cvref1: LCSC (none) -> C85979
- M1, M2: LCSC (none) -> C5334421
- Rcomp1: LCSC (none) -> C273789
- Rt1: LCSC (none) -> C844171
- Rvrefb1: LCSC (none) -> C165742
- Rvreft1: LCSC (none) -> C844784
Changed lines of the file:
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@@
+      (effects (font (size 1.27 1.27)) hide)
+    )
+    (property "LCSC" "C2842861" (id 4) (at 241.3 105.41 90)
       (effects (font (size 1.27 1.27)) hide)
     )
@@
     (property "Datasheet" "SIR180DP-T1-RE3" (id 3) (at 254 72.39 0)
       (effects (font (size 1.524 1.524)))
+    )
+    (property "LCSC" "C5334421" (id 4) (at 228.6 68.58 0)
+      (effects (font (size 1.27 1.27)) hide)
     )
     (pin "1")
@@
       (effects (font (size 1.27 1.27)) hide)
     )
+    (property "LCSC" "C85979" (id 4) (at 101.6 113.03 90)
+      (effects (font (size 1.27 1.27)) hide)
+    )
     (pin "1")
     (pin "2")
@@
     )
     (property "Datasheet" "~" (id 3) (at 106.68 120.65 0)
+      (effects (font (size 1.27 1.27)) hide)
+    )
+    (property "LCSC" "C165742" (id 4) (at 106.68 120.65 0)
       (effects (font (size 1.27 1.27)) hide)
     )
@@
       (effects (font (size 1.27 1.27)) hide)
     )
+    (property "LCSC" "C77093" (id 4) (at 241.3 132.08 90)
+      (effects (font (size 1.27 1.27)) hide)
+    )
     (pin "1")
     (pin "2")
@@
       (effects (font (size 1.27 1.27)) hide)
     )
+    (property "LCSC" "C77093" (id 4) (at 241.3 128.27 90)
+      (effects (font (size 1.27 1.27)) hide)
+    )
     (pin "1")
     (pin "2")
@@
       (effects (font (size 1.27 1.27)) hide)
     )
+    (property "LCSC" "C77093" (id 4) (at 241.3 151.13 90)
+      (effects (font (size 1.27 1.27)) hide)
+    )
     (pin "1")
     (pin "2")
@@
       (effects (font (size 1.27 1.27)) hide)
     )
+    (property "LCSC" "C92759" (id 4) (at 110.49 50.8 0)
+      (effects (font (size 1.27 1.27)) hide)
+    )
     (pin "1")
     (pin "2")
@@
     )
     (property "Datasheet" "~" (id 3) (at 106.68 115.57 0)
+      (effects (font (size 1.27 1.27)) hide)
+    )
+    (property "LCSC" "C844784" (id 4) (at 106.68 115.57 0)
       (effects (font (size 1.27 1.27)) hide)
     )
@@
       (effects (font (size 1.27 1.27)) hide)
     )
+    (property "LCSC" "C77093" (id 4) (at 241.3 147.32 90)
+      (effects (font (size 1.27 1.27)) hide)
+    )
     (pin "1")
     (pin "2")
@@
       (effects (font (size 1.27 1.27)) hide)
     )
+    (property "LCSC" "C92759" (id 4) (at 185.42 72.39 90)
+      (effects (font (size 1.27 1.27)) hide)
+    )
     (pin "1")
     (pin "2")
@@
     (property "Datasheet" "SIR180DP-T1-RE3" (id 3) (at 240.03 91.44 0)
       (effects (font (size 1.524 1.524)))
+    )
+    (property "LCSC" "C5334421" (id 4) (at 214.63 87.63 0)
+      (effects (font (size 1.27 1.27)) hide)
     )
     (pin "1")
@@
     )
     (property "Datasheet" "~" (id 3) (at 241.3 143.51 0)
+      (effects (font (size 1.27 1.27)) hide)
+    )
+    (property "LCSC" "C77093" (id 4) (at 241.3 143.51 90)
       (effects (font (size 1.27 1.27)) hide)
     )
@@
       (effects (font (size 1.27 1.27)) hide)
     )
+    (property "LCSC" "C2172920" (id 4) (at 97.79 50.8 0)
+      (effects (font (size 1.27 1.27)) hide)
+    )
     (pin "1")
     (pin "2")
@@
       (effects (font (size 1.27 1.27)) hide)
     )
+    (property "LCSC" "C77093" (id 4) (at 87.63 50.8 0)
+      (effects (font (size 1.27 1.27)) hide)
+    )
     (pin "1")
     (pin "2")
@@
       (effects (font (size 1.27 1.27)) hide)
     )
+    (property "LCSC" "C273789" (id 4) (at 105.41 97.79 90)
+      (effects (font (size 1.27 1.27)) hide)
+    )
     (pin "1")
     (pin "2")
@@
       (effects (font (size 1.27 1.27)) hide)
     )
+    (property "LCSC" "C77093" (id 4) (at 241.3 139.7 90)
+      (effects (font (size 1.27 1.27)) hide)
+    )
     (pin "1")
     (pin "2")
@@
     )
     (property "Datasheet" "~" (id 3) (at 77.47 50.8 0)
+      (effects (font (size 1.27 1.27)) hide)
+    )
+    (property "LCSC" "C77093" (id 4) (at 77.47 50.8 0)
       (effects (font (size 1.27 1.27)) hide)
     )
@@
       (effects (font (size 1.27 1.27)) hide)
     )
+    (property "LCSC" "C77093" (id 4) (at 241.3 154.94 90)
+      (effects (font (size 1.27 1.27)) hide)
+    )
     (pin "1")
     (pin "2")
@@
       (effects (font (size 1.27 1.27)) hide)
     )
+    (property "LCSC" "C107111" (id 4) (at 95.25 88.9 90)
+      (effects (font (size 1.27 1.27)) hide)
+    )
     (pin "1")
     (pin "2")
@@
       (effects (font (size 1.27 1.27)) hide)
     )
+    (property "LCSC" "C844171" (id 4) (at 111.76 82.55 90)
+      (effects (font (size 1.27 1.27)) hide)
+    )
     (pin "1")
     (pin "2")
@@
       (effects (font (size 1.27 1.27)) hide)
     )
+    (property "LCSC" "C77093" (id 4) (at 241.3 135.89 90)
+      (effects (font (size 1.27 1.27)) hide)
+    )

Commit message: updated from reviews
- changed capacitor
- changed output capacitors
- moved a bunch of stuff around and filled in a lot of copper area
Parts:
- removed Cout1, Cout2: 270u, Capacitor_SMD:C_0603_1608Metric, symbol Device:C_Small
- removed L1: 2.2u, inductor:HCMA1707-330-R, symbol Inductor:HCMA1707-330-R
- added Cout1, Cout2: 270u, 270u_cap:CAP_EEHZS1H271UP, symbol 270u_cap:EEHZS1H271UP
- added L1: 2.2, inductor2.2:IHLP6767GZER2R2M51, symbol Inductor2.2:IHLP6767GZER2R2M51
Connections:
- net GND: now also Cout1.2, Cout2.2
- net Vout: now also Cout1.1, Cout2.1
- net at Cbst1.2, M1.5, M1.6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: now also L1.1
- net at Rsense1.2, U1.2 (CSN): now also L1.2

Commit message: updated mosfets on high power 12V
Parts:
- removed M2: 60V, n-MOS:SIR826ADP-T1-GE3, symbol N-MOS:SIR826ADP-T1-GE3
- added M2: CSD18540Q5B, M2:TRANS_CSD18540Q5B, symbol M2:CSD18540Q5B
- M1: footprint n-MOS:SIR826ADP-T1-GE3 -> M1:TRANS_NVMFS5834NLWFT1G
Connections:
- net Vout: now also M2.5, M2.6, M2.7, M2.8
- net at Cbst1.2, L1.1, M1.5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: now also M2.1, M2.2, M2.3
- net at U1.5 (HO): now also M2.4
Changed lines of the file:
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@@
   (junction (at 227.33 77.47) (diameter 0) (color 0 0 0 0)
   )
-  (junction (at 236.22 58.42) (diameter 0) (color 0 0 0 0)
-  )
-  (junction (at 236.22 73.66) (diameter 0) (color 0 0 0 0)
-  )
   (junction (at 187.96 77.47) (diameter 0) (color 0 0 0 0)
   )
@@
   (junction (at 238.76 120.65) (diameter 0) (color 0 0 0 0)
   )
-  (junction (at 233.68 73.66) (diameter 0) (color 0 0 0 0)
-  )
   (junction (at 243.84 132.08) (diameter 0) (color 0 0 0 0)
   )
   (junction (at 238.76 151.13) (diameter 0) (color 0 0 0 0)
   )
-  (junction (at 241.3 58.42) (diameter 0) (color 0 0 0 0)
-  )
   (junction (at 243.84 128.27) (diameter 0) (color 0 0 0 0)
   )
@@
   (junction (at 246.38 114.3) (diameter 0) (color 0 0 0 0)
   )
-  (junction (at 238.76 58.42) (diameter 0) (color 0 0 0 0)
-  )
   (junction (at 238.76 139.7) (diameter 0) (color 0 0 0 0)
   )
@@
     (stroke (width 0) (type default) (color 0 0 0 0))
   )
-  (wire (pts (xy 241.3 58.42) (xy 246.38 58.42))
-    (stroke (width 0) (type default) (color 0 0 0 0))
-  )
   (wire (pts (xy 222.25 92.71) (xy 222.25 97.79))
     (stroke (width 0) (type default) (color 0 0 0 0))
@@
     (stroke (width 0) (type default) (color 0 0 0 0))
   )
-  (wire (pts (xy 228.6 68.58) (xy 194.31 68.58))
+  (wire (pts (xy 194.31 71.12) (xy 233.68 71.12))
     (stroke (width 0) (type default) (color 0 0 0 0))
   )
@@
     (stroke (width 0) (type default) (color 0 0 0 0))
   )
-  (wire (pts (xy 236.22 58.42) (xy 238.76 58.42))
-    (stroke (width 0) (type default) (color 0 0 0 0))
-  )
   (wire (pts (xy 77.47 74.93) (xy 77.47 129.54))
     (stroke (width 0) (type default) (color 0 0 0 0))
@@
     (stroke (width 0) (type default) (color 0 0 0 0))
   )
-  (wire (pts (xy 233.68 58.42) (xy 236.22 58.42))
-    (stroke (width 0) (type default) (color 0 0 0 0))
-  )
-  (wire (pts (xy 236.22 73.66) (xy 238.76 73.66))
-    (stroke (width 0) (type default) (color 0 0 0 0))
-  )
   (wire (pts (xy 238.76 147.32) (xy 238.76 151.13))
     (stroke (width 0) (type default) (color 0 0 0 0))
@@
     (stroke (width 0) (type default) (color 0 0 0 0))
   )
-  (wire (pts (xy 238.76 58.42) (xy 241.3 58.42))
-    (stroke (width 0) (type default) (color 0 0 0 0))
-  )
   (wire (pts (xy 187.96 77.47) (xy 210.82 77.47))
     (stroke (width 0) (type default) (color 0 0 0 0))
@@
     (stroke (width 0) (type default) (color 0 0 0 0))
   )
-  (wire (pts (xy 233.68 73.66) (xy 227.33 73.66))
-    (stroke (width 0) (type default) (color 0 0 0 0))
-  )
   (wire (pts (xy 96.52 123.19) (xy 96.52 113.03))
     (stroke (width 0) (type default) (color 0 0 0 0))
   )
-  (wire (pts (xy 233.68 73.66) (xy 236.22 73.66))
+  (wire (pts (xy 227.33 73.66) (xy 238.76 73.66))
     (stroke (width 0) (type default) (color 0 0 0 0))
   )
@@
     (stroke (width 0) (type default) (color 0 0 0 0))
   )
+  (wire (pts (xy 238.76 58.42) (xy 246.38 58.42))
+    (stroke (width 0) (type default) (color 0 0 0 0))
+  )
   (wire (pts (xy 246.38 120.65) (xy 246.38 128.27))
     (stroke (width 0) (type default) (color 0 0 0 0))
@@
     (stroke (width 0) (type default) (color 0 0 0 0))
   )
-  (wire (pts (xy 194.31 68.58) (xy 194.31 80.01))
+  (wire (pts (xy 194.31 71.12) (xy 194.31 80.01))
     (stroke (width 0) (type default) (color 0 0 0 0))
   )
@@
   )
   (wire (pts (xy 222.25 92.71) (xy 224.79 92.71))
+    (stroke (width 0) (type default) (color 0 0 0 0))
+  )
+  (wire (pts (xy 238.76 58.42) (xy 238.76 63.5))
     (stroke (width 0) (type default) (color 0 0 0 0))
   )
@@
     (pin "2")
   )
-  (symbol (lib_id "N-MOS:SIR826ADP-T1-GE3") (at 228.6 68.58 0) (unit 1)
-    (in_bom yes) (on_board yes)
-    (property "Reference" "M2" (id 0) (at 242.57 64.77 0)
-      (effects (font (size 1.524 1.524)) (justify left))
-    )
-    (property "Value" "60V" (id 1) (at 242.57 68.58 0)
-      (effects (font (size 1.524 1.524)) (justify left))
-    )
-    (property "Footprint" "n-MOS:SIR826ADP-T1-GE3" (id 2) (at 240.03 72.644 0)
-      (effects (font (size 1.524 1.524)) hide)
-    )
-    (property "Datasheet" "SIR180DP-T1-RE3" (id 3) (at 254 72.39 0)
-      (effects (font (size 1.524 1.524)))
-    )
-    (property "LCSC" "C5334421" (id 4) (at 228.6 68.58 0)
-      (effects (font (size 1.27 1.27)) hide)
-    )
-    (pin "1")
-    (pin "2")
-    (pin "3")
-    (pin "4")
-    (pin "5")
-    (pin "6")
-    (pin "7")
-    (pin "8")
-  )
   (symbol (lib_id "Device:C_Small") (at 101.6 113.03 90) (unit 1)
     (in_bom yes) (on_board yes) (fields_autoplaced)
@@
       (effects (font (size 1.524 1.524)) (justify left))
     )
-    (property "Footprint" "n-MOS:SIR826ADP-T1-GE3" (id 2) (at 226.06 91.694 0)
+    (property "Footprint" "M1:TRANS_NVMFS5834NLWFT1G" (id 2) (at 226.06 91.694 0)
       (effects (font (size 1.524 1.524)) hide)
     )
-    (property "Datasheet" "SIR180DP-T1-RE3" (id 3) (at 240.03 91.44 0)
+    (property "Datasheet" "NTMFS5C673NLT1G" (id 3) (at 240.03 91.44 0)
       (effects (font (size 1.524 1.524)))
     )
@@
     (pin "2")
   )
+  (symbol (lib_id "M2:CSD18540Q5B") (at 236.22 68.58 0) (unit 1)
+    (in_bom yes) (on_board yes) (fields_autoplaced)
+    (property "Reference" "M2" (id 0) (at 241.3 67.3099 0)
+      (effects (font (size 1.27 1.27)) (justify left))
+    )
+    (property "Value" "CSD18540Q5B" (id 1) (at 241.3 69.8499 0)
+      (effects (font (size 1.27 1.27)) (justify left))
+    )
+    (property "Footprint" "M2:TRANS_CSD18540Q5B" (id 2) (at 236.22 68.58 0)
+      (effects (font (size 1.27 1.27)) (justify bottom) hide)
+    )
+    (property "Datasheet" "" (id 3) (at 236.22 68.58 0)
+      (effects (font (size 1.27 1.27)) hide)
+    )
+    (property "MANUFACTURER" "Texas Instruments" (id 4) (at 236.22 68.58 0)
+      (effects (font (size 1.27 1.27)) (justify bottom) hide)
+    )
+    (property "PARTREV" "B" (id 5) (at 236.22 68.58 0)
+      (effects (font (size 1.27 1.27)) (justify bottom) hide)
+    )
+    (property "STANDARD" "Manufacturer recommendations" (id 6) (at 236.22 68.58 0)
+      (effects (font (size 1.27 1.27)) (justify bottom) hide)
+    )
+    (property "MAXIMUM_PACKAGE_HEIGHT" "1.05mm" (id 7) (at 236.22 68.58 0)
+      (effects (font (size 1.27 1.27)) (justify bottom) hide)
+    )
+    (pin "1")
+    (pin "2")
+    (pin "3")
+    (pin "4")
+    (pin "5")
+    (pin "6")
+    (pin "7")
+    (pin "8")
+  )
   (symbol (lib_id "power:GND") (at 181.61 115.57 90) (unit 1)
     (in_bom yes) (on_board yes) (fields_autoplaced)
@@
     )
     (path "/64391f12-acdd-4367-a4b2-5a471753d256"
-      (reference "M1") (unit 1) (value "60V") (footprint "n-MOS:SIR826ADP-T1-GE3")
-    )
-    (path "/06205616-782e-4f6d-8aba-a8fbdc766e75"
-      (reference "M2") (unit 1) (value "60V") (footprint "n-MOS:SIR826ADP-T1-GE3")
+      (reference "M1") (unit 1) (value "60V") (footprint "M1:TRANS_NVMFS5834NLWFT1G")
+    )
+    (path "/8eae0b44-4011-424d-acfe-3d644836614d"
+      (reference "M2") (unit 1) (value "CSD18540Q5B") (footprint "M2:TRANS_CSD18540Q5B")
     )
     (path "/ae518527-1660-4dba-8f0e-16d0914f5f97"

Commit message: add review notes
Parts:
- L1: value 2.2 -> 2.2u
Changed lines of the file:
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@@
       (effects (font (size 1.524 1.524)))
     )
-    (property "Value" "2.2" (id 1) (at 203.2 96.52 0)
+    (property "Value" "2.2u" (id 1) (at 203.2 96.52 0)
       (effects (font (size 1.524 1.524)))
     )
@@
     )
     (path "/cf998664-74b5-4732-a6f2-8ca78b745bd5"
-      (reference "L1") (unit 1) (value "2.2") (footprint "inductor2.2:IHLP6767GZER2R2M51")
+      (reference "L1") (unit 1) (value "2.2u") (footprint "inductor2.2:IHLP6767GZER2R2M51")
     )
     (path "/64391f12-acdd-4367-a4b2-5a471753d256"
